File: PCB/Mainboard/ADS1115.kicad_sch (KiCad schematic)
At the start: 1 part, among them J4 Conn_01x10_Pin

Commit message: First rev is done
Parts:
- J4: value Conn_01x10_Pin -> ADS1115
Changed lines of the file:
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@@
 			)
 		)
-		(property "Value" "Conn_01x10_Pin"
+		(property "Value" "ADS1115"
 			(at 131.445 85.09 0)
 			(effects
