File: PCB/Mainboard/AS7265x.kicad_sch (KiCad schematic)
At the start: 1 part, among them J2 Conn_01x06_Pin

Commit message: First rev is done
Parts:
- J2: value Conn_01x06_Pin -> AS7265X
Changed lines of the file:
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@@
 		(fields_autoplaced yes)
 		(property "Reference" "J2"
-			(at 141.605 105.41 0)
+			(at 143.51 92.7099 0)
 			(effects
 				(font
 					(size 1.27 1.27)
 				)
+				(justify right)
 			)
 		)
-		(property "Value" "Conn_01x06_Pin"
-			(at 141.605 102.87 0)
+		(property "Value" "AS7265X"
+			(at 143.51 95.2499 0)
 			(effects
 				(font
 					(size 1.27 1.27)
 				)
+				(justify right)
 			)
 		)
