File: PCB/Mainboard/GPSModule.kicad_sch (KiCad schematic)
At the start: 1 part, among them J1 Conn_GPS

Commit message: First rev is done
Parts:
- J1: value Conn_GPS -> GPS
Connections:
- net +3.3V renamed VCC
Changed lines of the file:
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@@
-	(wire
-		(pts
-			(xy 132.08 106.68) (xy 132.08 105.41)
-		)
-		(stroke
-			(width 0)
-			(type default)
-		)
-	)
 	(wire
 		(pts
@@
 		(shape input)
 		(at 134.62 106.68 90)
+		(fields_autoplaced yes)
+		(effects
+			(font
+				(size 1.27 1.27)
+			)
+			(justify left)
+		)
+	)
+	(hierarchical_label "VCC"
+		(shape input)
+		(at 132.08 106.68 90)
 		(fields_autoplaced yes)
 		(effects
@@
 	)
 	(symbol
-		(lib_id "power:+3.3V")
-		(at 132.08 105.41 0)
-		(unit 1)
-		(exclude_from_sim no)
-		(in_bom yes)
-		(on_board yes)
-		(dnp no)
-		(fields_autoplaced yes)
-		(property "Reference" "#PWR01"
-			(at 132.08 109.22 0)
-			(effects
-				(font
-					(size 1.27 1.27)
-				)
-				(hide yes)
-			)
-		)
-		(property "Value" "+3.3V"
-			(at 132.08 100.33 0)
-			(effects
-				(font
-					(size 1.27 1.27)
-				)
-			)
-		)
-		(property "Footprint" ""
-			(at 132.08 105.41 0)
-			(effects
-				(font
-					(size 1.27 1.27)
-				)
-				(hide yes)
-			)
-		)
-		(property "Datasheet" ""
-			(at 132.08 105.41 0)
-			(effects
-				(font
-					(size 1.27 1.27)
-				)
-				(hide yes)
-			)
-		)
-		(property "Description" "Power symbol creates a global label with name \"+3.3V\""
-			(at 132.08 105.41 0)
-			(effects
-				(font
-					(size 1.27 1.27)
-				)
-				(hide yes)
-			)
-		)
-		(pin "1"
-		)
-		(instances
-			(project "Mainboard"
-				(path "/2e068214-66f3-41bd-beea-f3af3145335c/a232a830-9c14-48b1-81a5-d9272c439a92"
-					(reference "#PWR01")
-					(unit 1)
-				)
-				(path "/2e068214-66f3-41bd-beea-f3af3145335c/870c4703-c4cd-4d8b-9509-4e4f0c7e7c0f"
-					(reference "#PWR09")
-					(unit 1)
-				)
-			)
-		)
-	)
-	(symbol
 		(lib_id "Connector:Conn_01x04_Pin")
 		(at 134.62 111.76 90)
@@
 		(fields_autoplaced yes)
 		(property "Reference" "J1"
-			(at 135.89 116.84 90)
+			(at 135.89 114.3 90)
 			(effects
 				(font
@@
 			)
 		)
-		(property "Value" "Conn_GPS"
-			(at 135.89 114.3 90)
+		(property "Value" "GPS"
+			(at 135.89 116.84 90)
 			(effects
 				(font
