File: PCB/Mainboard/GsmModule.kicad_sch (KiCad schematic)
At the start: 3 parts, among them U4 SIM800L-CORE

Commit message: updated some resitor values
Parts:
- R1: value 47K -> 1k
- R2: value 220K -> 10k
Changed lines of the file:
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@@
 (kicad_sch
-	(version 20231120)
+	(version 20250114)
 	(generator "eeschema")
-	(generator_version "8.0")
+	(generator_version "9.0")
 	(paper "A4")
 	(junction
@@
 		(shape input)
 		(at 124.46 104.14 180)
-		(fields_autoplaced yes)
 		(effects
 			(font
@@
 		(shape input)
 		(at 104.14 101.6 180)
-		(fields_autoplaced yes)
 		(effects
 			(font
@@
 		(shape input)
 		(at 124.46 99.06 180)
-		(fields_autoplaced yes)
 		(effects
 			(font
@@
 		(shape input)
 		(at 148.59 96.52 0)
-		(fields_autoplaced yes)
 		(effects
 			(font
@@
 			)
 		)
-		(property "Value" "47K"
+		(property "Value" "1k"
 			(at 109.22 97.79 90)
 			(effects
@@
 			)
 		)
-		(property "Value" "220K"
+		(property "Value" "10k"
 			(at 116.84 107.9499 0)
 			(effects
