File: PCB/Mainboard/SdCard.kicad_sch (KiCad schematic)
At the start: 1 part, among them J7 Conn_01x06_Pin

Commit message: First rev is done
Parts:
- J7: value Conn_01x06_Pin -> SD-Card
Changed lines of the file:
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@@
 			)
 		)
-		(property "Value" "Conn_01x06_Pin"
+		(property "Value" "SD-Card"
 			(at 136.525 96.52 0)
 			(effects
